Commit message: made it work in ros2 but cannot control yet

File: go1_description/xacro/depthCamera.xacro (robot description, xacro)
@@ -17,5 +17,5 @@
             <origin xyz="0 0 0" rpy="0 0 0"/>
             <geometry>
-                <mesh filename="package://meshes/depthCamera.dae" scale="1 1 1"/>
+                <mesh filename="file://$(find go1_description)/meshes/depthCamera.dae" scale="1 1 1"/>
             </geometry>
             </visual>

File: go1_description/xacro/gazebo.xacro (robot description, xacro)
@@ -2,10 +2,10 @@
 <robot>
     <!-- ros_control plugin -->
-    <gazebo>
+    <!-- <gazebo>
         <plugin name="gazebo_ros_control" filename="libgazebo_ros_control.so">
             <robotNamespace>/go1_gazebo</robotNamespace>
             <robotSimType>gazebo_ros_control/DefaultRobotHWSim</robotSimType>
         </plugin>
-    </gazebo>
+    </gazebo> -->
     <!-- Show the trajectory of trunk center. -->
     <gazebo>
@@ -19,22 +19,11 @@
         </plugin>
     </gazebo>
-    <!-- Show the trajectory of foot. You can add another trajectory about another foot. -->
     <!-- <gazebo>
-        <plugin name="3dplot" filename="libLinkPlot3DPlugin.so">
-            <frequency>100</frequency>
-            <plot>
-                <link>FL_foot</link>
-                <pose>0 0 0 0 0 0</pose>
-                <material>Gazebo/Green</material>
-            </plot>
+        <plugin filename="libgazebo_ros_force.so" name="gazebo_ros_force">
+            <body_name>trunk</body_name>
+            <topic_name>/apply_force/trunk</topic_name>
         </plugin>
     </gazebo> -->
-    <gazebo>
-        <plugin filename="libgazebo_ros_force.so" name="gazebo_ros_force">
-            <bodyName>trunk</bodyName>
-            <topicName>/apply_force/trunk</topicName>
-        </plugin>
-    </gazebo>
-    <gazebo reference="imu_link">
+    <!-- <gazebo reference="imu_link">
         <gravity>true</gravity>
         <sensor name="imu_sensor" type="imu">
@@ -54,76 +43,26 @@
             <pose>0 0 0 0 0 0</pose>
         </sensor>
-    </gazebo>
-    <!-- Depth camera -->
-    <!-- <gazebo>
-        <plugin name="camera_plugin" filename="libgazebo_ros_openni_kinect.so">
-            <baseline>0.025</baseline>
+    </gazebo> -->
+    <gazebo reference="imu_link">
+        <sensor name="imu_controller" type="imu">
             <always_on>true</always_on>
-            <updateRate>0.0</updateRate>
-            <cameraName>unitree_camera_left</cameraName>
-            <frameName>depthCamera_link_left</frameName>
-            <imageTopicName>rgb/imageRaw_left</imageTopicName>
-            <depthImageTopicName>depth/imageRaw_left</depthImageTopicName>
-            <pointCloudTopicName>depth/points_left</pointCloudTopicName>
-            <cameraInfoTopicName>rgb/cameraInfo_left</cameraInfoTopicName>
-            <depthImageCameraInfoTopicName>depth/cameraInfo_left</depthImageCameraInfoTopicName>
-            <pointCloudCutoff>0.1</pointCloudCutoff>
-            <pointCloudCutoffMax>1.5</pointCloudCutoffMax>
-            <distortionK1>0.0</distortionK1>
-            <distortionK2>0.0</distortionK2>
-            <distortionK3>0.0</distortionK3>
-            <distortionT1>0.0</distortionT1>
-            <distortionT2>0.0</distortionT2>
-            <CxPrime>0.0</CxPrime>
-            <Cx>0.0045</Cx>
-            <Cy>0.0039</Cy>
-            <focalLength>0.004</focalLength>
-            <hackBaseline>0.0</hackBaseline>
-        </plugin>
-    </gazebo> -->
-    <!-- <gazebo reference="depthCamera_link_left">
-        <sensor name="unitree_camera_left" type="depth_camera">
-            <update_rate>16</update_rate>
-            <always_on>true</always_on>
-            <visualize>true</visualize>
-            <camera>
-                <horizontal_fov>2.094</horizontal_fov>
-                <image>
-                    <width>928</width>
-                    <height>800</height>
-                    <format>R8G8B8</format>
-                </image>
-                <depth_camera></depth_camera>
-                <clip>
-                    <near>0.1</near>
-                    <far>100</far>
-                </clip>
-            </camera>
-            <plugin name="camera_plugin" filename="libgazebo_ros_openni_kinect.so">
-                <baseline>0.025</baseline>
-                <always_on>true</always_on>
-                <updateRate>0.0</updateRate>
-                <cameraName>unitree_camera_left</cameraName>
-                <frameName>depthCamera_link_left</frameName>
-                <imageTopicName>rgb/imageRaw_left</imageTopicName>
-                <depthImageTopicName>depth/imageRaw_left</depthImageTopicName>
-                <pointCloudTopicName>depth/points_left</pointCloudTopicName>
-                <cameraInfoTopicName>rgb/cameraInfo_left</cameraInfoTopicName>
-                <depthImageCameraInfoTopicName>depth/cameraInfo_left</depthImageCameraInfoTopicName>
-                <pointCloudCutoff>0.1</pointCloudCutoff>
-                <pointCloudCutoffMax>1.5</pointCloudCutoffMax>
-                <distortionK1>0.0</distortionK1>
-                <distortionK2>0.0</distortionK2>
-                <distortionK3>0.0</distortionK3>
-                <distortionT1>0.0</distortionT1>
-                <distortionT2>0.0</distortionT2>
-                <CxPrime>0.0</CxPrime>
-                <Cx>0.0045</Cx>
-                <Cy>0.0039</Cy>
-                <focalLength>0.004</focalLength>
-                <hackBaseline>0.0</hackBaseline>
-            </plugin>
-        </sensor>
-    </gazebo> -->
+            <update_rate>1000</update_rate>
+            <plugin name="gazebo_ros_imu_sensor" filename="libgazebo_ros_imu_sensor.so">
+                <ros>
+                    <namespace>/imu</namespace>
+                    <argument>~/out:=data</argument>
+                </ros>
+                <!-- <updateRate>50.0</updateRate>
+                <bodyName>imu_link</bodyName>
+                <topicName>imu/data</topicName>
+                <accelDrift>0.005 0.005 0.005</accelDrift>
+                <accelGaussianNoise>0.005 0.005 0.005</accelGaussianNoise>
+                <rateDrift>0.005 0.005 0.005 </rateDrift>
+                <rateGaussianNoise>0.005 0.005 0.005 </rateGaussianNoise>
+                <headingDrift>0.005</headingDrift>
+                <headingGaussianNoise>0.005</headingGaussianNoise> -->
+            </plugin>
+        </sensor>
+    </gazebo>
   <gazebo reference="depthCamera_link_left">
     <sensor name="camera_link_camera" type="depth">
@@ -168,5 +107,5 @@
   </gazebo>
     <!-- Foot contacts. -->
-    <gazebo reference="FR_calf">
+    <!-- <gazebo reference="FR_calf">
         <sensor name="FR_foot_contact" type="contact">
         <update_rate>100</update_rate>
@@ -203,7 +142,7 @@
         </contact>
         </sensor>
-    </gazebo>
+    </gazebo> -->
     <!-- Visualization of Foot contacts. -->
-    <gazebo reference="FR_foot">
+    <!-- <gazebo reference="FR_foot">
         <visual>
             <plugin name="drawForcePlugin" filename="libunitreeDrawForcePlugin.so">
@@ -232,5 +171,5 @@
             </plugin>
         </visual>
-    </gazebo>
+    </gazebo> -->
     <gazebo reference="base">
         <material>Gazebo/Green</material>
@@ -253,9 +192,9 @@
         <material>Gazebo/Red</material>
     </gazebo>
-    <!-- FL leg -->
+    <!-- fl leg -->
     <gazebo reference="FL_hip">
         <mu1>0.2</mu1>
         <mu2>0.2</mu2>
-        <material>Gazebo/DarkGrey</material>
+        <material>Gazebo/Gray</material>
     </gazebo>
     <gazebo reference="FL_thigh">
@@ -263,5 +202,5 @@
         <mu2>0.2</mu2>
         <self_collide>1</self_collide>
-        <material>Gazebo/DarkGrey</material>
+        <material>Gazebo/White</material>
         <kp  value="1000000.0"/>
         <kd  value="1.0"/>
@@ -271,4 +210,5 @@
         <mu2>0.2</mu2>
         <self_collide>1</self_collide>
+        <material>Gazebo/White</material>
     </gazebo>
     <gazebo reference="FL_foot">
@@ -276,13 +216,13 @@
         <mu2>0.6</mu2>
         <self_collide>1</self_collide>
-        <material>Gazebo/DarkGrey</material>
-        <kp  value="1000000.0"/>
-        <kd  value="1.0"/>
-    </gazebo>
-    <!-- FR leg -->
+        <material>Gazebo/White</material>
+        <kp  value="1000000.0"/>
+        <kd  value="1.0"/>
+    </gazebo>
+    <!-- fr leg -->
     <gazebo reference="FR_hip">
         <mu1>0.2</mu1>
         <mu2>0.2</mu2>
-        <material>Gazebo/DarkGrey</material>
+        <material>Gazebo/Gray</material>
     </gazebo>
     <gazebo reference="FR_thigh">
@@ -290,5 +230,5 @@
         <mu2>0.2</mu2>
         <self_collide>1</self_collide>
-        <material>Gazebo/DarkGrey</material>
+        <material>Gazebo/White</material>
         <kp  value="1000000.0"/>
         <kd  value="1.0"/>
@@ -298,4 +238,5 @@
         <mu2>0.2</mu2>
         <self_collide>1</self_collide>
+        <material>Gazebo/White</material>
     </gazebo>
     <gazebo reference="FR_foot">
@@ -303,5 +244,5 @@
         <mu2>0.6</mu2>
         <self_collide>1</self_collide>
-        <material>Gazebo/DarkGrey</material>
+        <material>Gazebo/White</material>
         <kp  value="1000000.0"/>
         <kd  value="1.0"/>
@@ -311,5 +252,5 @@
         <mu1>0.2</mu1>
         <mu2>0.2</mu2>
-        <material>Gazebo/DarkGrey</material>
+        <material>Gazebo/Gray</material>
     </gazebo>
     <gazebo reference="RL_thigh">
@@ -317,5 +258,5 @@
         <mu2>0.2</mu2>
         <self_collide>1</self_collide>
-        <material>Gazebo/DarkGrey</material>
+        <material>Gazebo/White</material>
         <kp  value="1000000.0"/>
         <kd  value="1.0"/>
@@ -330,5 +271,5 @@
         <mu2>0.6</mu2>
         <self_collide>1</self_collide>
-        <material>Gazebo/DarkGrey</material>
+        <material>Gazebo/White</material>
         <kp  value="1000000.0"/>
         <kd  value="1.0"/>
@@ -338,5 +279,5 @@
         <mu1>0.2</mu1>
         <mu2>0.2</mu2>
-        <material>Gazebo/DarkGrey</material>
+        <material>Gazebo/Gray</material>
     </gazebo>
     <gazebo reference="RR_thigh">
@@ -344,5 +285,5 @@
         <mu2>0.2</mu2>
         <self_collide>1</self_collide>
-        <material>Gazebo/DarkGrey</material>
+        <material>Gazebo/White</material>
         <kp  value="1000000.0"/>
         <kd  value="1.0"/>
@@ -352,4 +293,5 @@
         <mu2>0.2</mu2>
         <self_collide>1</self_collide>
+        <material>Gazebo/White</material>
     </gazebo>
     <gazebo reference="RR_foot">
@@ -357,7 +299,30 @@
         <mu2>0.6</mu2>
         <self_collide>1</self_collide>
-        <material>Gazebo/DarkGrey</material>
-        <kp  value="1000000.0"/>
-        <kd  value="1.0"/>
+        <material>Gazebo/White</material>
+        <kp  value="1000000.0"/>
+        <kd  value="1.0"/>
+    </gazebo>
+    <gazebo>
+      <plugin name="p3d_base_controller" filename="libgazebo_ros_p3d.so">
+        <ros>
+            <argument>odom:=odom/ground_truth</argument>
+        </ros>
+        <body_name>trunk</body_name>
+        <frame_name>world</frame_name>
+        <update_rate>10.0</update_rate>
+        <xyz_offset>0 0 0</xyz_offset>
+        <rpy_offset>0 0 0</rpy_offset>
+        <gaussian_noise>0.01</gaussian_noise>
+    </plugin>
+    </gazebo>
+    <!-- <gazebo>
+        <plugin filename="libgazebo_ros2_control.so" name="gazebo_ros2_control">
+        <parameters>$(find go1_description)/config/ros_control/ros_control.yaml</parameters>
+      </plugin>
+    </gazebo> -->
+    <gazebo>
+        <plugin filename="libgazebo_ros2_control.so" name="gazebo_ros2_control">
+        <parameters>$(find go1_description)/config/ros_control/go1_controller.yaml</parameters>
+      </plugin>
     </gazebo>
 </robot>

File: go1_description/xacro/leg2.xacro (robot description, xacro)
@@ -256,17 +256,20 @@
             </hardware>
             <joint name="${name}_hip_joint">
-                <command_interface name="effort" />
+                <command_interface name="position" />
                 <state_interface name="position"/>
                 <state_interface name="velocity" />
+                <state_interface name="effort" />
             </joint>
             <joint name="${name}_thigh_joint">
-                <command_interface name="effort" />
+                <command_interface name="position" />
                 <state_interface name="position" />
                 <state_interface name="velocity" />
+                <state_interface name="effort" />
             </joint>
             <joint name="${name}_calf_joint">
-                <command_interface name="effort" />
+                <command_interface name="position" />
                 <state_interface name="position" />
                 <state_interface name="velocity" />
+                <state_interface name="effort" />
             </joint>
         </ros2_control>

File: go1_description/xacro/robot.xacro (robot description, xacro)
@@ -4,5 +4,5 @@
     <xacro:include filename="$(find go1_description)/xacro/const.xacro"/>
     <xacro:include filename="$(find go1_description)/xacro/materials.xacro"/>
-    <xacro:include filename="$(find go1_description)/xacro/leg.xacro"/>
+    <xacro:include filename="$(find go1_description)/xacro/leg2.xacro"/>
     <!-- <xacro:include filename="$(find go1_description)/xacro/stairs.xacro"/> -->
     <xacro:include filename="$(find go1_description)/xacro/gazebo.xacro"/>
@@ -39,5 +39,5 @@
             <origin rpy="0 0 0" xyz="0 0 0"/>
             <geometry>
-                <mesh filename="package://meshes/trunk.dae" scale="1 1 1"/>
+                <mesh filename="file://$(find go1_description)/meshes/trunk.dae" scale="1 1 1"/>
             </geometry>
             <!-- <material name="orange"/> -->
@@ -83,5 +83,5 @@
         </collision>
     </link>
-    <xacro:leg name="FR" mirror="-1" mirror_dae= "False" front_hind="1"  front_hind_dae="True"  />
+    <xacro:leg name="FR" mirror="-1" mirror_dae="False"  front_hind="1"  front_hind_dae="True"  />
     <xacro:leg name="FL" mirror="1"  mirror_dae="True"   front_hind="1"  front_hind_dae="True"  />
     <xacro:leg name="RR" mirror="-1" mirror_dae="False"  front_hind="-1" front_hind_dae="False" />

File: go1_description/xacro/ultraSound.xacro (robot description, xacro)
@@ -17,5 +17,5 @@
             <origin xyz="0 0 0" rpy="0 0 0"/>
             <geometry>
-                <mesh filename="package://meshes/ultraSound.dae" scale="1 1 1"/>
+                <mesh filename="file://$(find go1_description)/meshes/ultraSound.dae" scale="1 1 1"/>
             </geometry>
             <material name="black"/>
